File: hardware/RFM69CW_BOB.brd (EAGLE design)
At the start: 27.9 x 20.3 mm, 11 parts, among them U1 RFM69HCW

Commit message: HCW BOB to 1.0, CW BOB to 0.1
Parts:
- U1: value RFM69HCW -> RFM69CW; device mike-temp:RFM69HCW-XXXS2 -> mike-temp:RFM69CW-XXXS2
- turned U1 to 180 degrees
Connections:
- removed net DIO4: JP3.4, U1.12
- net 3.3V: now also U1.2; no longer U1.13
- net ANT: now also U1.1; no longer U1.9
- net DIO0: now also U1.9; no longer U1.14
- net DIO1: now also U1.11; no longer U1.15
- net DIO2: now also U1.10; no longer U1.16
- net DIO3: now also U1.4; no longer U1.11
- net DIO5: now also U1.12; no longer U1.7
- net GND: now also U1.14, U1.3; no longer U1.1, U1.10, U1.8
- net MISO: now also U1.8; no longer U1.2
- net MOSI: now also U1.5; no longer U1.3
- net NSS: now also U1.7; no longer U1.5
- net RESET: now also U1.13; no longer U1.6
- net SCK: now also U1.6; no longer U1.4
Routing:
- net NSS: track 5.61 -> 22.7 mm, vias 0 -> 1
- net DIO1: track 6.29 -> 23.4 mm, vias 0 -> 1
- net SCK: track 5.84 -> 22.0 mm, vias 0 -> 1
- net MOSI: track 6.06 -> 21.5 mm, vias 0 -> 1
- net DIO0: track 23.5 -> 12.5 mm, vias 1 -> 0
- net DIO2: track 13.4 -> 23.1 mm
- net DIO3: track 14.9 -> 6.25 mm, vias 1 -> 0
- net RESET: track 5.39 -> 13.2 mm, vias 0 -> 1
- net DIO4: track 5.61 -> 0.00 mm
- net 3.3V: track 35.1 -> 31.1 mm
- net DIO5: track 21.3 -> 20.4 mm
Other:
- board text added: "RFM69CW"
- board text added: "V01"
- board text removed: "4"
- board text removed: "DIO4"
- board text removed: "RFM69HCW"
- board text removed: "V10"
