File: hardware/RFM69HCW_BOB.sch (EAGLE design)
At the start: 11 parts, among them U1 RFM69HCW

Commit message: Added fiducials to HCW BOB, initial example code
Parts:
- added FID1, FID2: FIDUCIAL1X2, SparkFun-Aesthetics:FIDUCIAL1X2
Changed lines of the file:
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@@
 <?xml version="1.0" encoding="utf-8"?>
 <!DOCTYPE eagle SYSTEM "eagle.dtd">
-<eagle version="6.4">
+<eagle version="6.5.0">
 <drawing>
 <settings>
@@
 <part name="JP2" library="mike-temp" deviceset="M01" device="SMDNS"/>
 <part name="JP3" library="mike-temp" deviceset="M05" device="_ROUNDONLY_NOSILK"/>
+<part name="FID1" library="SparkFun-Aesthetics" deviceset="FIDUCIAL" device="1X2"/>
+<part name="FID2" library="SparkFun-Aesthetics" deviceset="FIDUCIAL" device="1X2"/>
 </parts>
 <sheets>
@@
 <instance part="JP2" gate="G$1" x="160.02" y="127" rot="R180"/>
 <instance part="JP3" gate="G$1" x="160.02" y="111.76" rot="R180"/>
+<instance part="FID1" gate="G$1" x="241.3" y="25.4"/>
+<instance part="FID2" gate="G$1" x="246.38" y="25.4"/>
 </instances>
 <busses>

Commit message: Changed capacitor, removed C variant
Changed C1 to CAP-9824 (10uF ceramic for better transient response)
Removed RFM69C (low power) for future BOB
Parts:
- removed JP8: (no value), mike-temp:M021X02_NO_SILK
- added JP4: (no value), mike-temp:M05_ROUNDONLY_NOSILK
- C1: device SparkFun-Capacitors:10UF-16V-10%(TANT) -> SparkFun-Capacitors:10UF50V20%(1210)
- JP1: device mike-temp:M05_ROUNDONLY_NOSILK -> mike-temp:M021X02_NO_SILK
- JP2: device mike-temp:M01SMDNS -> mike-temp:M05_ROUNDONLY_NOSILK
- JP3: device mike-temp:M05_ROUNDONLY_NOSILK -> mike-temp:M01SMDNS
- renumbered JP7 to JP5
Connections:
- net 3.3V: now also C1.1, JP1.1; no longer C1.+, JP8.1
- net DIO0: now also JP3.1; no longer JP2.1
- net DIO1: now also JP4.1; no longer JP3.1
- net DIO2: now also JP4.2; no longer JP3.2
- net DIO3: now also JP4.3; no longer JP3.3
- net DIO4: now also JP4.4; no longer JP3.4
- net DIO5: now also JP4.5; no longer JP3.5
- net GND: now also C1.2, JP1.2; no longer C1.-, JP8.2
- net MISO: now also JP2.1; no longer JP1.1
- net MOSI: now also JP2.2; no longer JP1.2
- net NSS: now also JP2.4; no longer JP1.4
- net RESET: now also JP2.5; no longer JP1.5
- net SCK: now also JP2.3; no longer JP1.3
Changed lines of the file:
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@@
 <part name="FRAME1" library="SparkFun-Aesthetics" deviceset="FRAME-LETTER" device=""/>
 <part name="C2" library="SparkFun-Capacitors" deviceset="0.1UF-25V(+80/-20%)(0603)" device="" value="0.1uF"/>
-<part name="C1" library="SparkFun-Capacitors" deviceset="10UF-16V-10%(TANT)" device="" value="10uF"/>
 <part name="SUPPLY1" library="SparkFun-Aesthetics" deviceset="3.3V" device=""/>
 <part name="SUPPLY2" library="SparkFun-Aesthetics" deviceset="3.3V" device=""/>
@@
 <part name="LOGO1" library="SparkFun-Aesthetics" deviceset="SFE_LOGO_NAME" device=".1_INCH" value="SFE_LOGO_NAME.1_INCH"/>
 <part name="LOGO2" library="SparkFun-Aesthetics" deviceset="OSHW-LOGO" device="S"/>
-<part name="JP7" library="mike-temp" deviceset="M03" device="_ROUND_ONLY_NO_SILK" value="ANTENNA"/>
-<part name="JP8" library="mike-temp" deviceset="M02" device="1X02_NO_SILK"/>
+<part name="JP5" library="mike-temp" deviceset="M03" device="_ROUND_ONLY_NO_SILK" value="ANTENNA"/>
+<part name="JP1" library="mike-temp" deviceset="M02" device="1X02_NO_SILK"/>
 <part name="SUPPLY4" library="SparkFun-Aesthetics" deviceset="3.3V" device=""/>
 <part name="GND4" library="SparkFun-Aesthetics" deviceset="GND" device=""/>
-<part name="JP1" library="mike-temp" deviceset="M05" device="_ROUNDONLY_NOSILK"/>
-<part name="JP2" library="mike-temp" deviceset="M01" device="SMDNS"/>
-<part name="JP3" library="mike-temp" deviceset="M05" device="_ROUNDONLY_NOSILK"/>
+<part name="JP2" library="mike-temp" deviceset="M05" device="_ROUNDONLY_NOSILK"/>
+<part name="JP3" library="mike-temp" deviceset="M01" device="SMDNS"/>
+<part name="JP4" library="mike-temp" deviceset="M05" device="_ROUNDONLY_NOSILK"/>
 <part name="FID1" library="SparkFun-Aesthetics" deviceset="FIDUCIAL" device="1X2"/>
 <part name="FID2" library="SparkFun-Aesthetics" deviceset="FIDUCIAL" device="1X2"/>
+<part name="C1" library="SparkFun-Capacitors" deviceset="10UF50V20%(1210)" device="" value="10uF"/>
 </parts>
 <sheets>
@@
 <instance part="FRAME1" gate="G$2" x="147.32" y="0"/>
 <instance part="C2" gate="G$1" x="68.58" y="106.68"/>
-<instance part="C1" gate="G$1" x="58.42" y="109.22"/>
 <instance part="SUPPLY1" gate="G$1" x="58.42" y="116.84"/>
 <instance part="SUPPLY2" gate="G$1" x="68.58" y="116.84"/>
@@
 <instance part="LOGO1" gate="G$1" x="147.32" y="35.56"/>
 <instance part="LOGO2" gate="G$1" x="233.68" y="45.72"/>
-<instance part="JP7" gate="G$1" x="160.02" y="91.44" rot="R180"/>
-<instance part="JP8" gate="G$1" x="83.82" y="127" rot="MR180"/>
+<instance part="JP5" gate="G$1" x="160.02" y="91.44" rot="R180"/>
+<instance part="JP1" gate="G$1" x="83.82" y="127" rot="MR180"/>
 <instance part="SUPPLY4" gate="G$1" x="93.98" y="129.54"/>
 <instance part="GND4" gate="1" x="93.98" y="119.38"/>
-<instance part="JP1" gate="G$1" x="83.82" y="106.68" rot="MR180"/>
-<instance part="JP2" gate="G$1" x="160.02" y="127" rot="R180"/>
-<instance part="JP3" gate="G$1" x="160.02" y="111.76" rot="R180"/>
+<instance part="JP2" gate="G$1" x="83.82" y="106.68" rot="MR180"/>
+<instance part="JP3" gate="G$1" x="160.02" y="127" rot="R180"/>
+<instance part="JP4" gate="G$1" x="160.02" y="111.76" rot="R180"/>
 <instance part="FID1" gate="G$1" x="241.3" y="25.4"/>
 <instance part="FID2" gate="G$1" x="246.38" y="25.4"/>
+<instance part="C1" gate="G$1" x="58.42" y="106.68"/>
 </instances>
 <busses>
@@
 <wire x1="137.16" y1="96.52" x2="137.16" y2="88.9" width="0.1524" layer="91"/>
 <wire x1="134.62" y1="96.52" x2="137.16" y2="96.52" width="0.1524" layer="91"/>
-<pinref part="JP7" gate="G$1" pin="1"/>
+<pinref part="JP5" gate="G$1" pin="1"/>
 <wire x1="134.62" y1="101.6" x2="142.24" y2="101.6" width="0.1524" layer="91"/>
 <wire x1="142.24" y1="101.6" x2="142.24" y2="93.98" width="0.1524" layer="91"/>
 <wire x1="142.24" y1="93.98" x2="152.4" y2="93.98" width="0.1524" layer="91"/>
-<pinref part="JP7" gate="G$1" pin="3"/>
+<pinref part="JP5" gate="G$1" pin="3"/>
 <wire x1="137.16" y1="88.9" x2="142.24" y2="88.9" width="0.1524" layer="91"/>
 <label x="144.78" y="93.98" size="1.778" layer="95"/>
@@
 </segment>
 <segment>
-<pinref part="C1" gate="G$1" pin="-"/>
 <pinref part="GND1" gate="1" pin="GND"/>
 <wire x1="58.42" y1="99.06" x2="58.42" y2="104.14" width="0.1524" layer="91"/>
+<pinref part="C1" gate="G$1" pin="2"/>
 </segment>
 <segment>
@@
 </segment>
 <segment>
-<pinref part="JP8" gate="G$1" pin="2"/>
+<pinref part="JP1" gate="G$1" pin="2"/>
 <wire x1="91.44" y1="124.46" x2="93.98" y2="124.46" width="0.1524" layer="91"/>
 <wire x1="93.98" y1="124.46" x2="93.98" y2="121.92" width="0.1524" layer="91"/>
@@
 </segment>
 <segment>
-<pinref part="C1" gate="G$1" pin="+"/>
 <pinref part="SUPPLY1" gate="G$1" pin="3.3V"/>
 <wire x1="58.42" y1="116.84" x2="58.42" y2="111.76" width="0.1524" layer="91"/>
-</segment>
-<segment>
-<pinref part="JP8" gate="G$1" pin="1"/>
+<pinref part="C1" gate="G$1" pin="1"/>
+</segment>
+<segment>
+<pinref part="JP1" gate="G$1" pin="1"/>
 <wire x1="91.44" y1="127" x2="93.98" y2="127" width="0.1524" layer="91"/>
 <wire x1="93.98" y1="127" x2="93.98" y2="129.54" width="0.1524" layer="91"/>
@@
 <wire x1="137.16" y1="119.38" x2="134.62" y2="119.38" width="0.1524" layer="91"/>
 <label x="144.78" y="127" size="1.778" layer="95"/>
-<pinref part="JP2" gate="G$1" pin="1"/>
+<pinref part="JP3" gate="G$1" pin="1"/>
 </segment>
 </net>
@@
 <wire x1="152.4" y1="116.84" x2="134.62" y2="116.84" width="0.1524" layer="91"/>
 <label x="144.78" y="116.84" size="1.778" layer="95"/>
-<pinref part="JP3" gate="G$1" pin="1"/>
+<pinref part="JP4" gate="G$1" pin="1"/>
 </segment>
 </net>
@@
 <wire x1="152.4" y1="114.3" x2="134.62" y2="114.3" width="0.1524" layer="91"/>
 <label x="144.78" y="114.3" size="1.778" layer="95"/>
-<pinref part="JP3" gate="G$1" pin="2"/>
+<pinref part="JP4" gate="G$1" pin="2"/>
 </segment>
 </net>
@@
 <wire x1="152.4" y1="111.76" x2="134.62" y2="111.76" width="0.1524" layer="91"/>
 <label x="144.78" y="111.76" size="1.778" layer="95"/>
-<pinref part="JP3" gate="G$1" pin="3"/>
+<pinref part="JP4" gate="G$1" pin="3"/>
 </segment>
 </net>
@@
 <wire x1="91.44" y1="111.76" x2="104.14" y2="111.76" width="0.1524" layer="91"/>
 <label x="91.44" y="111.76" size="1.778" layer="95"/>
-<pinref part="JP1" gate="G$1" pin="1"/>
+<pinref part="JP2" gate="G$1" pin="1"/>
 </segment>
 </net>
@@
 <wire x1="91.44" y1="109.22" x2="104.14" y2="109.22" width="0.1524" layer="91"/>
 <label x="91.44" y="109.22" size="1.778" layer="95"/>
-<pinref part="JP1" gate="G$1" pin="2"/>
+<pinref part="JP2" gate="G$1" pin="2"/>
 </segment>
 </net>
@@
 <wire x1="91.44" y1="106.68" x2="104.14" y2="106.68" width="0.1524" layer="91"/>
 <label x="91.44" y="106.68" size="1.778" layer="95"/>
-<pinref part="JP1" gate="G$1" pin="3"/>
+<pinref part="JP2" gate="G$1" pin="3"/>
 </segment>
 </net>
@@
 <wire x1="91.44" y1="104.14" x2="104.14" y2="104.14" width="0.1524" layer="91"/>
 <label x="91.44" y="104.14" size="1.778" layer="95"/>
-<pinref part="JP1" gate="G$1" pin="4"/>
+<pinref part="JP2" gate="G$1" pin="4"/>
 </segment>
 </net>
@@
 <wire x1="101.6" y1="96.52" x2="104.14" y2="96.52" width="0.1524" layer="91"/>
 <label x="91.44" y="101.6" size="1.778" layer="95"/>
-<pinref part="JP1" gate="G$1" pin="5"/>
+<pinref part="JP2" gate="G$1" pin="5"/>
 <wire x1="91.44" y1="101.6" x2="101.6" y2="101.6" width="0.1524" layer="91"/>
 <wire x1="101.6" y1="101.6" x2="101.6" y2="96.52" width="0.1524" layer="91"/>
@@
 <net name="ANT" class="0">
 <segment>
-<pinref part="JP7" gate="G$1" pin="2"/>
+<pinref part="JP5" gate="G$1" pin="2"/>
 <pinref part="U1" gate="G$1" pin="ANT"/>
 <wire x1="152.4" y1="91.44" x2="139.7" y2="91.44" width="0.1524" layer="91"/>
@@
 <wire x1="134.62" y1="106.68" x2="152.4" y2="106.68" width="0.1524" layer="91"/>
 <label x="144.78" y="106.68" size="1.778" layer="95"/>
-<pinref part="JP3" gate="G$1" pin="5"/>
+<pinref part="JP4" gate="G$1" pin="5"/>
 </segment>
 </net>
@@
 <wire x1="152.4" y1="109.22" x2="134.62" y2="109.22" width="0.1524" layer="91"/>
 <label x="144.78" y="109.22" size="1.778" layer="95"/>
-<pinref part="JP3" gate="G$1" pin="4"/>
-</segment>
-</net>
+<pinref part="JP4" gate="G$1" pin="4"/>
+</segment>
+</net>

Commit message: Changed version to 1.0 for reds
Other:
- note added: "1.0"
- note removed: "01"
Changed lines of the file:
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@@
 <plain>
 <text x="172.72" y="7.62" size="2.54" layer="94">M Grusin</text>
-<text x="241.3" y="7.62" size="2.54" layer="94">01</text>
+<text x="241.3" y="7.62" size="2.54" layer="94">1.0</text>
 <text x="2.54" y="5.08" size="2.54" layer="94">Note: Mark board with frequency of installed module</text>
 <text x="167.64" y="83.82" size="2.54" layer="94">Antenna length (1/4 wave)
